Commit message: Step 19: front camera publishing /camera/image_raw with optical frame TF

File: ros2_ws/src/security_robot_webots/resource/security_robot_description.urdf (robot description, URDF)
Before this commit: robot security_robot, 7 links, 6 joints
Links:
- added link camera_link; visual box size=0.02 0.04 0.03
- added link camera_optical_link
Joints:
- added joint camera_joint: type fixed, parent base_link, child camera_link, origin xyz=0.1 0 0.13 rpy=0 0 0
- added joint camera_optical_joint: type fixed, parent camera_link, child camera_optical_link, origin xyz=0 0 0 rpy=-1.5708 0 -1.5708

Commit message: Realistic scale: 8x6 m office world, scaled robot with camera mast, recalibrated odometry

File: ros2_ws/src/security_robot_webots/resource/security_robot_description.urdf (robot description, URDF)
Before this commit: robot security_robot, 9 links, 8 joints
Links:
- added link mast_link; visual cylinder length=0.68 radius=0.02
- link base_link: geometry visual box size=0.44 0.38 0.18
- link camera_link: geometry visual box size=0.04 0.08 0.05
- link front_caster: geometry visual sphere radius=0.03
- link left_wheel: geometry visual cylinder length=0.04 radius=0.08
- link lidar_link: geometry visual cylinder length=0.05 radius=0.05
- link rear_caster: geometry visual sphere radius=0.03
- link right_wheel: geometry visual cylinder length=0.04 radius=0.08
Joints:
- added joint mast_joint: type fixed, parent base_link, child mast_link, origin xyz=-0.15 0 0.55 rpy=0 0 0
- joint camera_joint: origin xyz=0.1 0 0.13 rpy=0 0 0 -> xyz=-0.15 0 0.92 rpy=0 0 0
- joint front_caster_joint: origin xyz=0.08 0 0.015 rpy=0 0 0 -> xyz=0.18 0 0.03 rpy=0 0 0
- joint left_wheel_joint: origin xyz=0 0.09 0.03 rpy=0 0 0 -> xyz=0 0.22 0.08 rpy=0 0 0
- joint lidar_joint: origin xyz=0 0 0.09 rpy=0 0 0 -> xyz=0 0 0.25 rpy=0 0 0
- joint rear_caster_joint: origin xyz=-0.08 0 0.015 rpy=0 0 0 -> xyz=-0.18 0 0.03 rpy=0 0 0
- joint right_wheel_joint: origin xyz=0 -0.09 0.03 rpy=0 0 0 -> xyz=0 -0.22 0.08 rpy=0 0 0

Commit message: IMU: gyro fused into odometry via complementary filter in the driver; EKF config kept for hardware

File: ros2_ws/src/security_robot_webots/resource/security_robot_description.urdf (robot description, URDF)
Before this commit: robot security_robot, 10 links, 9 joints
Links:
- added link imu_link
Joints:
- added joint imu_joint: type fixed, parent base_link, child imu_link, origin xyz=0 0 0.12 rpy=0 0 0
